File: can_fet_egt_sd_v2.sch (KiCad schematic (older format))
At the start: 21 parts, among them J10 Molex_Micro-Fit_3.0_43045-060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, J14 microSD_HC_Wuerth_693072010801, J20 Conn_02x05_Odd_Even-Connector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, J21 Soldering PAD for 12V_MREL, J30 Conn_02x05_Odd_Even-Connector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, J40 CONN_Molex, P1104 CONN_Sparkfun, Q1 BTS3028, U1101 MAX31855KASA, U5 TJA1051T-3

Commit message: Add files via upload
Parts:
- U1101: footprint Package_SO:SO-8_5.3x6.2mm_P1.27mm -> Package_SO:SOIC-8_3.9x4.9mm_P1.27mm
Changed lines of the file:
@@
 F 0 "U6" H 5625 4500 60  0000 C CNN
 F 1 "MAX31855KASA" H 5625 4000 60  0000 C CNN
-F 2 "Package_SO:SO-8_5.3x6.2mm_P1.27mm" V 805 2450 60  0001 C CNN
+F 2 "Package_SO:SOIC-8_3.9x4.9mm_P1.27mm" V 805 2450 60  0001 C CNN
 F 3 "" H 5625 4250 60  0001 C CNN
 F 4 "DALLAS SEMI,MAX31855KASA+	" V 805 2450 60  0001 C CNN "MFG,MFG#"

Commit message: Add files via upload
Parts:
- removed J40: CONN_Molex, Connector_Molex:Molex_Micro-Fit_3.0_43045-0200_2x01_P3.00mm_Horizontal, symbol Connector:Conn_01x02_Male
- added C27: 100nF, Capacitor_SMD:C_0603_1608Metric, symbol Device:C
- F1: footprint Resistor_SMD:R_1206_3216Metric -> Resistor_SMD:R_2816_7142Metric
- J10: value Molex_Micro-Fit_3.0_43045-0601_43045-0612 -> Molex_Micro-Fit_3.0_43045-0800_43045-0812; footprint Connector_Molex:Molex_Micro-Fit_3.0_43045-0600_2x03_P3.00mm_Horizontal -> Connector_Molex:Molex_Micro-Fit_3.0_43045-0800_2x04_P3.00mm_Horizontal; symbol mre_addon_v2-rescue:Conn_Molex_02x03-wideband_controller_mre-rescue-wideband_controller_mre-rescue -> mre_addon_v2-rescue:Conn_Molex_02x04-wideband_controller_mre-rescue-wideband_controller_mre-rescue
Other:
- moved on the sheet: C26, F1, J20, J21, J30, J41
