File: mcu_adc_mre_wbo2_v2x.sch (KiCad schematic (older format))
At the start: 51 parts, among them J1 TC2030, J2 Conn_01x06_Male, J3 Conn_01x03_Male, SW1 SW_Push, U1 STM32F072CBUx, U2 MCP6004, U3 AD8628, U4 REF3033

Commit message: Add files via upload
Parts:
- added C33, C36: 2.2u, Capacitor_SMD:C_0603_1608Metric, symbol Device:C
- added C34: 100n, Capacitor_SMD:C_0402_1005Metric, symbol Device:C
- added C35: 1u, Capacitor_SMD:C_0603_1608Metric, symbol Device:C
- added R27, R36: 10k, Resistor_SMD:R_0402_1005Metric, symbol Device:R
- added R28, R34: 3.3k, Resistor_SMD:R_0603_1608Metric, symbol Device:R
- added R31, R35: 330R, Resistor_SMD:R_0603_1608Metric, symbol Device:R
- added R32, R37: 82k, Resistor_SMD:R_0603_1608Metric, symbol Device:R
- added R33, R38: 160k, Resistor_SMD:R_0603_1608Metric, symbol Device:R
- added U5, U7: MCP6002-xSN, Package_SO:SO-8_3.9x4.9mm_P1.27mm, symbol wideband_controller-rescue:MCP6002-xSN-Amplifier_Operational
Connections:
- net +5V: now also C34.1, C35.1, R27.2, U7.8 (V+)
- net GND: now also C33.2, C34.2, C35.2, C36.2, R33.1, R36.1, R38.1, U7.4 (V-)
- net PWMout2: now reaches U1.27 (PB14)
- net PWMout2: now also R34.1
- net PWMout1: now reaches U1.28 (PB15)
- net PWMout1: now also R28.1
- new net: R35.1, R37.2, U5.1
- new net: R37.1, R38.2, U5.2 (-)
- new net: C36.1, R34.2, U5.3 (+)
- new net: R32.1, R33.2, U5.6 (-)
- new net: R31.1, R32.2, U5.7
- new net: C33.1, R28.2, U5.5 (+)
- new net Vout1: R27.1, R31.2
- new net Vout2: R35.2, R36.2
- no-connect marks 22 -> 20
Other:
- note added: "1.524x gain"
- note added: "2x Buffered outputs"
- moved on the sheet: C12, C13, C2, C5, C6, J1, J2, J3, R19, R20, R21, R22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
