File: mre_addon_v2.kicad_pcb (KiCad board)
At the start: 2 copper layers, 80.6 x 48.4 mm, 82 parts, among them J1 TC2030, J10 Molex_Micro-Fit_3.0_43045-060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, J10 Molex_Micro-Fit_3.0_43045-061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, J15 microSD_HC_Wuerth_693072010801, J15x MICRO-SDCARD-CONNECTOR-330006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, J2 Conn_01x06_Male, J20 Conn_02x05_Odd_Even-Connector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, J21 Soldering PAD for 12V_MREL, J3 Conn_01x03_Male, J30 Conn_02x05_Odd_Even-Connector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

Commit message: Add files via upload
Parts:
- U6: footprint Package_SO:SO-8_5.3x6.2mm_P1.27mm -> Package_SO:SO-8_3.9x4.9mm_P1.27mm
- moved U6 1.15 mm to (80.0, 139.8)
- moved C16 0.20 mm to (114.8, 131.0)
- moved J3 0.06 mm to (94.7, 133.2)
Routing:
- net /can_fet_egt_sd_v2/PA15: track 77.7 -> 76.1 mm
- net /can_fet_egt_sd_v2/PC10: track 98.1 -> 99.2 mm
- net /can_fet_egt_sd_v2/PC11: track 95.7 -> 96.5 mm

Commit message: Add files via upload
Parts:
- added C27: 100nF, Capacitor_SMD:C_0603_1608Metric, F.Cu at (135.8, 153.7)
- added C8: 100n, Capacitor_SMD:C_0603_1608Metric, F.Cu at (127.1, 153.8)
- F1: value R_2816_7142Metric -> Polyfuse 2A
- J10: value Molex_Micro-Fit_3.0_43045-0612_2x03_P3.00mm_Vertical -> Molex_Micro-Fit_3.0_43045-0812_2x04_P3.00mm_Vertical; footprint Connector_Molex:Molex_Micro-Fit_3.0_43045-0612_2x03_P3.00mm_Vertical -> Connector_Molex:Molex_Micro-Fit_3.0_43045-0812_2x04_P3.00mm_Vertical
- J10: value Molex_Micro-Fit_3.0_43045-0601_43045-0612 -> Molex_Micro-Fit_3.0_43045-0800_43045-0812; footprint Connector_Molex:Molex_Micro-Fit_3.0_43045-0600_2x03_P3.00mm_Horizontal -> Connector_Molex:Molex_Micro-Fit_3.0_43045-0800_2x04_P3.00mm_Horizontal
- U6: footprint Package_SO:SO-8_3.9x4.9mm_P1.27mm -> Package_SO:SOIC-8_3.9x4.9mm_P1.27mm
- moved C25 63.1 mm to (138.8, 157.8), turned to 270 degrees
- moved U6 57.4 mm to (134.3, 158.5), turned to 180 degrees
- moved J40x 36.0 mm to (50.1, 119.2)
- moved J40 34.5 mm to (50.0, 130.7)
- moved D2 19.5 mm to (124.0, 159.6), turned to 90 degrees
- moved D3 17.3 mm to (122.3, 159.6), turned to 90 degrees
- moved C7 3.26 mm to (120.2, 153.8)
- moved C9 3.26 mm to (118.5, 153.8)
- moved C17 3.26 mm to (125.4, 153.8)
- moved U4 3.12 mm to (122.8, 154.0)
- moved D3 3.10 mm to (114.4, 146.3)
- moved D2 3.10 mm to (114.4, 144.8)
- moved R32 3.10 mm to (134.2, 153.7)
- moved R33 3.02 mm to (132.8, 153.7)
- moved R34 3.00 mm to (131.2, 153.7)
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Connections:
- D2 pad 1: Net-(D2-Pad1) -> GND (x2)
- D2 pad 2: /mcu_adc_mre_wbo2_v2/LED_GREEN -> Net-(D2-Pad2) (x2)
- D3 pad 1: Net-(D3-Pad1) -> GND (x2)
- D3 pad 2: /mcu_adc_mre_wbo2_v2/LED_BLUE -> Net-(D3-Pad2) (x2)
- J10 pad 4: LSU_Ip -> /can_fet_egt_sd_v2/TCPL- (x2)
- J10 pad 5: /can_fet_egt_sd_v2/LSU_Heater- -> LSU_Ip (x2)
- J10 pad 6: LSU_Rtrim -> /can_fet_egt_sd_v2/LSU_Heater- (x2)
- J2 pad 2: /mcu_adc_mre_wbo2_v2/nRESET -> /mcu_adc_mre_wbo2_v2/SWCLK
- J2 pad 3: /mcu_adc_mre_wbo2_v2/SWCLK -> GND
- J2 pad 5: /mcu_adc_mre_wbo2_v2/SWO -> /mcu_adc_mre_wbo2_v2/nRESET
- J2 pad 6: GND -> /mcu_adc_mre_wbo2_v2/SWO
- R24 pad 1: GND -> Net-(D2-Pad2)
- R24 pad 2: Net-(D2-Pad1) -> /mcu_adc_mre_wbo2_v2/LED_GREEN
- R25 pad 1: GND -> Net-(D3-Pad2)
- R25 pad 2: Net-(D3-Pad1) -> /mcu_adc_mre_wbo2_v2/LED_BLUE
Routing:
- net /can_fet_egt_sd_v2/PA15: track 76.1 -> 26.3 mm, vias 2 -> 1
- net /can_fet_egt_sd_v2/PC10: track 99.2 -> 72.6 mm, vias 3 -> 1
- net /can_fet_egt_sd_v2/PC11: track 96.5 -> 75.4 mm
- net Net-(D2-Pad2): track 0.00 -> 20.4 mm, vias 0 -> 1
- net Net-(D3-Pad2): track 0.00 -> 18.7 mm, vias 0 -> 1
- net GND: track 98.1 -> 89.1 mm, vias 85 -> 82
- net heater_pwm: track 47.3 -> 43.6 mm
- net /mcu_adc_mre_wbo2_v2/SWCLK: track 33.4 -> 36.9 mm
- net +3.3V: track 249.8 -> 253.1 mm, vias 10 -> 11
- net /mcu_adc_mre_wbo2_v2/nRESET: track 34.0 -> 30.7 mm, vias 1 -> 2
- net VDDA: track 41.5 -> 38.7 mm
- net /mcu_adc_mre_wbo2_v2/Ip_sense: track 23.0 -> 20.3 mm
- net /mcu_adc_mre_wbo2_v2/SWO: track 8.96 -> 6.42 mm
- net /can_fet_egt_sd_v2/PC12: track 65.0 -> 67.5 mm, vias 3 -> 1
- net Net-(D1-Pad2): track 2.83 -> 5.09 mm
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Other:
- outline, holes or cut-outs redrawn
- board text added: "3.3V SWCLK GND SWDIO nRESET SWO"
- board text added: "J21"
- board text added: "K-Thermocouple"
- board text added: "SD Card CS# PIN - PB9 EGT Chip CS# PIN - PA15"
- board text added: "SWO nRESET SWDIO GND SWCLK 3.3V"
- board text added: "WBO2 controller by mck1117 PCB ver.2.3 by JRD McLAREN"
- board text added: "ver. 2.3"
- board text removed: "3.3V nRESET SWCLK SWDIO SWO GND"
- board text removed: "GND SWO SWDIO SWCLK nRESET 3.3V"
- board text removed: "K - Thermocouple"
- board text removed: "WBO2 controller by mck1117 PCB ver.2.2 by JRD McLAREN"
- board text removed: "ver. 2.2"

Commit message: Add files via upload
Parts:
- added J30: Conn_02x05_Odd_Even-Connector_Generic, Connector_PinHeader_2.54mm:PinHeader_2x05_P2.54mm_Vertical_SMD, B.Cu at (130.0, 167.1)
Connections:
- J40 pad 1: /can_fet_egt_sd_v2/TCPL+ -> (no net)
- J40 pad 2: /can_fet_egt_sd_v2/TCPL- -> (no net)
- J40x pad 1: /can_fet_egt_sd_v2/TCPL+ -> (no net)
- J40x pad 2: /can_fet_egt_sd_v2/TCPL- -> (no net)
Routing:
- net GND: track 89.1 -> 99.4 mm, vias 82 -> 84
- net /can_fet_egt_sd_v2/PC11: track 75.4 -> 74.5 mm
- net /can_fet_egt_sd_v2/PC10: track 72.6 -> 71.7 mm
