File: mre_addon_v2.kicad_pcb (KiCad board)
At the start: 2 copper layers, 80.6 x 48.4 mm, 85 parts, among them J1 TC2030, J10 Molex_Micro-Fit_3.0_43045-080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, J10 Molex_Micro-Fit_3.0_43045-081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, J15 microSD_HC_Wuerth_693072010801, J15x MICRO-SDCARD-CONNECTOR-330006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, J2 Conn_01x06_Male, J20 Conn_02x05_Odd_Even-Connector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, J21 Soldering PAD for 12V_MREL, J3 Conn_01x03_Male, J30 Conn_02x05_Odd_Even-Connector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

Commit message: Add files via upload
Parts:
- added F1: R_Axial_DIN0207_L6.3mm_D2.5mm_P10.16mm_Horizontal, Resistor_THT:R_Axial_DIN0207_L6.3mm_D2.5mm_P10.16mm_Horizontal, F.Cu at (151.1, 128.7)
- moved J40x 36.1 mm to (84.6, 129.9)
- moved J40 34.7 mm to (84.6, 129.9)
- moved J21 5.65 mm to (145.5, 128.2)
Routing:
- net /can_fet_egt_sd_v2/12V_MREL: track 9.52 -> 28.4 mm
- net GND: vias 84 -> 85

Commit message: Add files via upload
Parts:
- moved J40 0.07 mm to (84.5, 129.9)
- moved J40x 0.07 mm to (84.5, 129.9)
Other:
- outline, holes or cut-outs redrawn
Changed lines of the file:
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@@
     (mod_text_width 0.15)
     (pad_size 1.6 1.6)
-    (pad_drill 0.8)
+    (pad_drill 0)
     (pad_to_mask_clearance 0.051)
     (solder_mask_min_width 0.25)
@@
   )
   (module Connector_Molex:Molex_Micro-Fit_3.0_43045-0212_2x01_P3.00mm_Vertical (layer F.Cu)
-    (at 84.62 129.9 90)
+    (at 84.55 129.9 90)
     (descr "Molex Micro-Fit 3.0 Connector System, 43045-0212 (compatible alternatives: 43045-0213, 43045-0224), 1 Pins per row (http://www.molex.com/pdm_docs/sd/430450212_sd.pdf), generated with kicad-footprint-generator")
     (tags "connector Molex Micro-Fit_3.0 side entry")
@@
   )
   (module Connector_Molex:Molex_Micro-Fit_3.0_43045-0200_2x01_P3.00mm_Horizontal (layer F.Cu)
-    (at 84.62 129.9 90)
+    (at 84.55 129.9 90)
     (descr "Molex Micro-Fit 3.0 Connector System, 43045-0200 (alternative finishes: 43045-020x), 1 Pins per row (https://www.molex.com/pdm_docs/sd/430450201_sd.pdf), generated with kicad-footprint-generator")
     (tags "connector Molex Micro-Fit_3.0 horizontal")
@@
     (pad M12 thru_hole circle (at -38.7096 -9.6824 270) (size 1.6 1.6) (drill 1.15) (layers *.Cu *.Mask))
     (pad M13 thru_hole circle (at -38.7096 -12.2224 270) (size 1.6 1.6) (drill 1.15) (layers *.Cu *.Mask))
-    (pad M3 thru_hole rect (at -6.3246 -21.1124 270) (size 1.6 1.6) (drill 1.15) (layers *.Cu *.Mask))
-    (pad M4 thru_hole rect (at 5.7404 -21.1124 270) (size 1.6 1.6) (drill 1.15) (layers *.Cu *.Mask))
+    (pad "" connect rect (at -6.3246 -21.1124 270) (size 1.6 1.6) (layers B.Cu B.Mask))
+    (pad "" connect rect (at 5.7404 -21.1124 270) (size 1.6 1.6) (layers B.Cu B.Mask))
     (pad M21 thru_hole rect (at 38.7604 -7.1424 270) (size 1.6 1.6) (drill 1.15) (layers *.Cu *.Mask))
     (pad M22 thru_hole circle (at 38.7604 -9.6824 270) (size 1.6 1.6) (drill 1.15) (layers *.Cu *.Mask))
@@
   (gr_circle (center 98.4 147.05) (end 103.4 147.05) (layer B.SilkS) (width 0.12))
   (gr_circle (center 96.95 145) (end 101.95 145) (layer B.SilkS) (width 0.12))
-  (gr_line (start 111.6 169.3) (end 119.6 169.3) (layer Edge.Cuts) (width 0.12))
-  (gr_line (start 121.4 167.5) (end 121.4 163.3) (layer Edge.Cuts) (width 0.12))
-  (gr_line (start 109.8 163.3) (end 109.8 167.5) (layer Edge.Cuts) (width 0.12))
-  (gr_line (start 111.6 161.5) (end 119.6 161.5) (layer Edge.Cuts) (width 0.12))
-  (gr_arc (start 111.6 163.3) (end 111.6 161.5) (angle -90) (layer Edge.Cuts) (width 0.12))
+  (gr_line (start 111.5 170.3) (end 119.6 170.3) (layer Edge.Cuts) (width 0.12))
+  (gr_line (start 121.4 168.5) (end 121.4 163.3) (layer Edge.Cuts) (width 0.12))
+  (gr_line (start 109.7 163.3) (end 109.7 168.5) (layer Edge.Cuts) (width 0.12))
+  (gr_line (start 111.5 161.5) (end 119.6 161.5) (layer Edge.Cuts) (width 0.12))
+  (gr_arc (start 111.5 163.3) (end 111.5 161.5) (angle -90) (layer Edge.Cuts) (width 0.12))
   (gr_arc (start 119.6 163.3) (end 121.4 163.3) (angle -90) (layer Edge.Cuts) (width 0.12))
-  (gr_arc (start 111.6 167.5) (end 109.8 167.5) (angle -90) (layer Edge.Cuts) (width 0.12))
-  (gr_arc (start 119.6 167.5) (end 119.6 169.3) (angle -90) (layer Edge.Cuts) (width 0.12))
+  (gr_arc (start 111.5 168.5) (end 109.7 168.5) (angle -90) (layer Edge.Cuts) (width 0.12))
+  (gr_arc (start 119.6 168.5) (end 119.6 170.3) (angle -90) (layer Edge.Cuts) (width 0.12))
   (gr_line (start 98.4 147.6) (end 98.4 146.5) (layer B.SilkS) (width 0.12))
   (gr_line (start 97.85 147.05) (end 98.95 147.05) (layer B.SilkS) (width 0.12))

Commit message: Add files via upload
Routing:
- net GND: track 99.4 -> 105.1 mm
Other:
- outline, holes or cut-outs redrawn
Changed lines of the file:
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@@
   (general
     (thickness 1.6)
-    (drawings 76)
-    (tracks 931)
+    (drawings 81)
+    (tracks 938)
     (zones 0)
     (modules 86)
@@
   )
   (setup
-    (last_trace_width 0.25)
+    (last_trace_width 0.5)
     (user_trace_width 0.2)
     (user_trace_width 0.3)
@@
       (drillshape 0)
       (scaleselection 1)
-      (outputdirectory "gerbers/V2.3"))
+      (outputdirectory "gerbers/V2.3x"))
   )
   (net 0 "")
@@
     )
   )
+  (gr_line (start 109.8 172.4) (end 121.3 172.4) (layer Edge.Cuts) (width 0.3))
+  (gr_line (start 143.1 172.1) (end 152.6 163) (layer Edge.Cuts) (width 0.3))
+  (gr_line (start 87.5 172) (end 78 163) (layer Edge.Cuts) (width 0.3))
+  (gr_line (start 154 139.9) (end 154 129) (layer Edge.Cuts) (width 0.3))
+  (gr_line (start 76.6 145) (end 76.6 134) (layer Edge.Cuts) (width 0.3))
   (gr_text "SD Card CS# PIN - PB9\nEGT Chip CS# PIN - PA15" (at 118.7 144.85) (layer B.SilkS)
     (effects (font (size 1 1) (thickness 0.25)) (justify mirror))
@@
   (segment (start 136.620001 151.979999) (end 135.634999 151.979999) (width 0.3) (layer F.Cu) (net 1))
   (via (at 120.7 136.2) (size 0.6) (drill 0.3) (layers F.Cu B.Cu) (net 1))
+  (segment (start 98.21 165.785) (end 97.925 165.5) (width 0.5) (layer F.Cu) (net 1))
+  (segment (start 98.21 167.035) (end 98.21 165.785) (width 0.5) (layer F.Cu) (net 1))
+  (segment (start 98.21 168.285) (end 98.2 168.295) (width 0.5) (layer F.Cu) (net 1))
+  (segment (start 98.21 167.035) (end 98.21 168.285) (width 0.5) (layer F.Cu) (net 1))
+  (segment (start 97.668 158.369) (end 97.7 158.401) (width 0.5) (layer F.Cu) (net 1))
+  (segment (start 97.668 157.107) (end 97.668 158.369) (width 0.5) (layer F.Cu) (net 1))
+  (segment (start 97.668 157.107) (end 97.668 155.632) (width 0.5) (layer F.Cu) (net 1))
   (segment (start 122.4 132) (end 122.35 132.05) (width 0.25) (layer F.Cu) (net 2))
   (segment (start 126 127.4125) (end 127.6 127.4125) (width 0.25) (layer F.Cu) (net 2))
@@
   (segment (start 103.761478 137.25) (end 104.8375 137.25) (width 0.25) (layer F.Cu) (net 28))
   (segment (start 102.82501 136.313532) (end 103.761478 137.25) (width 0.25) (layer F.Cu) (net 28))
-  (segment (start 93.97 134.795) (end 94.47501 135.30001) (width 0.25) (layer F.Cu) (net 28))
-  (segment (start 90.875 134.795) (end 93.97 134.795) (width 0.25) (layer F.Cu) (net 28))
   (segment (start 102.27499 135.30001) (end 102.37503 135.30001) (width 0.25) (layer F.Cu) (net 28))
-  (segment (start 94.47501 135.30001) (end 102.27499 135.30001) (width 0.25) (layer F.Cu) (net 28))
   (segment (start 102.82502 136.313522) (end 102.82501 136.313532) (width 0.25) (layer F.Cu) (net 28))
   (segment (start 102.824981 135.524981) (end 102.82502 136.313522) (width 0.25) (layer F.Cu) (net 28))
   (segment (start 102.60001 135.30001) (end 102.824981 135.524981) (width 0.25) (layer F.Cu) (net 28))
   (segment (start 102.27499 135.30001) (end 102.60001 135.30001) (width 0.25) (layer F.Cu) (net 28))
+  (segment (start 92.4 134.8) (end 90.875 134.795) (width 0.25) (layer F.Cu) (net 28))
+  (segment (start 92.90001 135.30001) (end 92.4 134.8) (width 0.25) (layer F.Cu) (net 28))
+  (segment (start 102.27499 135.30001) (end 92.90001 135.30001) (width 0.25) (layer F.Cu) (net 28))
   (segment (start 117.074999 133.574999) (end 117.1 133.6) (width 0.25) (layer F.Cu) (net 35))
   (segment (start 113.337501 133.574999) (end 117.074999 133.574999) (width 0.25) (layer F.Cu) (net 35))

Commit message: Add files via upload
Parts:
- removed J40: CONN_Molex, Connector_Molex:Molex_Micro-Fit_3.0_43045-0200_2x01_P3.00mm_Horizontal
- removed J40x: Molex_Micro-Fit_3.0_43045-0212_2x01_P3.00mm_Vertical, Connector_Molex:Molex_Micro-Fit_3.0_43045-0212_2x01_P3.00mm_Vertical
- added ?: , , F.Cu at (90.0, 147.3)
- added ?: , , F.Cu at (88.8, 146.2)
- added C18: 18pF, Capacitor_SMD:C_0603_1608Metric, F.Cu at (117.0, 140.3)
- added C19: 18pF, Capacitor_SMD:C_0603_1608Metric, F.Cu at (117.0, 132.6)
- added H1: MountingHole_3.2mm_M3_Pad_Via, MountingHole:MountingHole_3.2mm_M3_Pad_Via, F.Cu at (88.5, 162.7)
- added H2: MountingHole_3.2mm_M3_Pad_Via, MountingHole:MountingHole_3.2mm_M3_Pad_Via, F.Cu at (142.2, 162.7)
- added J1: TC2030, rusefi_lib:Tag-Connect_TC2030-IDC-NL_2x03_P1.27mm_Vertical, B.Cu at (96.6, 129.0)
- added Y1: 8MHz, Crystal:Crystal_SMD_5032-2Pin_5.0x3.2mm, F.Cu at (117.2, 136.4)
- J10: value Molex_Micro-Fit_3.0_43045-0812_2x04_P3.00mm_Vertical -> Molex_Micro-Fit_3.0_43045-0800_43045-0812
- moved LOGO1 49.0 mm to (91.4, 169.1)
- moved C16 11.7 mm to (103.2, 130.8), turned to 180 degrees
- moved R4 8.40 mm to (129.4, 128.2)
- moved C4 8.40 mm to (127.8, 128.2), turned to 90 degrees
- moved R9 6.89 mm to (119.8, 128.2)
- moved C26 4.49 mm to (86.7, 133.2), turned to 180 degrees
- moved R8 4.06 mm to (121.5, 142.4)
- moved C1 2.95 mm to (124.7, 128.2), turned to 90 degrees
- moved J15x 2.75 mm to (100.8, 161.8)
- moved R12 2.25 mm to (123.0, 142.4)
- moved C3 2.25 mm to (124.7, 142.4)
- moved R10 2.25 mm to (126.2, 142.4)
- moved R11 2.20 mm to (127.8, 142.4)
- moved R14 2.20 mm to (129.4, 142.4)
- moved R6 2.15 mm to (128.9, 135.0)
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- renumbered U3 to U3x
Connections:
- J15 pad 1: Net-(J15-Pad1) -> unconnected-(J15-Pad1)
- J15 pad 8: Net-(J15-Pad8) -> unconnected-(J15-Pad8)
- U1 pad 14: Net-(U1-Pad14) -> unconnected-(U1-Pad14)
- U1 pad 15: Net-(U1-Pad15) -> unconnected-(U1-Pad15)
- U1 pad 18: Net-(U1-Pad18) -> unconnected-(U1-Pad18)
- U1 pad 2: Net-(U1-Pad2) -> unconnected-(U1-Pad2)
- U1 pad 20: Net-(U1-Pad20) -> unconnected-(U1-Pad20)
- U1 pad 21: Net-(U1-Pad21) -> unconnected-(U1-Pad21)
- U1 pad 22: Net-(U1-Pad22) -> unconnected-(U1-Pad22)
- U1 pad 25: Net-(U1-Pad25) -> unconnected-(U1-Pad25)
- U1 pad 26: Net-(U1-Pad26) -> unconnected-(U1-Pad26)
- U1 pad 27: Net-(U1-Pad27) -> unconnected-(U1-Pad27)
- U1 pad 28: Net-(U1-Pad28) -> unconnected-(U1-Pad28)
- U1 pad 3: Net-(U1-Pad3) -> unconnected-(U1-Pad3)
- U1 pad 38: Net-(U1-Pad38) -> unconnected-(U1-Pad38)
- U1 pad 39: Net-(U1-Pad39) -> unconnected-(U1-Pad39)
- U1 pad 4: Net-(U1-Pad4) -> unconnected-(U1-Pad4)
- U1 pad 40: Net-(U1-Pad40) -> unconnected-(U1-Pad40)
- U1 pad 45: Net-(U1-Pad45) -> unconnected-(U1-Pad45)
- U1 pad 46: Net-(U1-Pad46) -> unconnected-(U1-Pad46)
- U6 pad 8: Net-(U6-Pad8) -> unconnected-(U6-Pad8)
Routing:
- net /mcu_adc_mre_wbo2_v2/SWDIO: track 27.8 -> 47.1 mm
- net /mcu_adc_mre_wbo2_v2/SWCLK: track 36.9 -> 53.3 mm
- net Net-(R4-Pad2): track 27.2 -> 14.6 mm, vias 0 -> 2
- net GND: track 105.1 -> 94.5 mm, vias 85 -> 65
- net /mcu_adc_mre_wbo2_v2/nRESET: track 30.7 -> 41.0 mm
- net /mcu_adc_mre_wbo2_v2/Ip_dac: track 14.2 -> 22.7 mm
- net VDDA: track 38.7 -> 46.0 mm
- net Net-(C19-Pad2): track 0.00 -> 6.95 mm
- net Net-(C18-Pad2): track 0.00 -> 6.90 mm
- net /mcu_adc_mre_wbo2_v2/Ip_sense: track 20.3 -> 27.2 mm
- net Net-(R11-Pad2): track 11.5 -> 18.3 mm
- net /mcu_adc_mre_wbo2_v2/SWO: track 6.42 -> 13.1 mm
- net +5V: track 141.5 -> 147.8 mm
- net /can_fet_egt_sd_v2/PC11: track 74.5 -> 80.5 mm
- net /can_fet_egt_sd_v2/PB9: track 70.2 -> 75.7 mm
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Other:
- board size 80.6 x 48.4 mm -> 76.6 x 46.8 mm
- net class Default removed
- board text added: "H+"
- board text added: "H-"
- board text added: "MAX13054"
- board text added: "WBO2 controller by mck1117 PCB ver.2.5 by JRD McLAREN"
- board text added: "ver. 2.5"
- board text removed: "Heater+"
- board text removed: "Heater-"
- board text removed: "TJA1051T"
- board text removed: "WBO2 controller by mck1117 PCB ver.2.3 by JRD McLAREN"
- board text removed: "ver. 2.3"
