File: can_fet_egt_sd_v2.kicad_sch (KiCad schematic)
At the start: 21 parts, among them J10 Molex_Micro-Fit_3.0_43045-080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, J15 microSD_HC_Wuerth_693072010801, J20 Conn_02x05_Odd_Even-Connector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, J21 Soldering PAD for 12V_MREL, J30 Conn_02x05_Odd_Even-Connector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, J41 CONN_Sparkfun, Q1 BTS3028, U5 TJA1051T-3, U6 MAX31855KASA

Commit message: V2.5 with OPAmp
Parts:
- added C28: 100n, Capacitor_SMD:C_0603_1608Metric, symbol Device:C
- added J40: Molex_Micro-Fit_3.0_43045-0200_2x01_P3.00mm_Horiz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, Molex_Micro-Fit_3.0_43045-0200_2x01_P3.00mm_Horizontal, symbol Connector_Generic:Conn_01x02
- added R35, R40: 160k, Resistor_SMD:R_0603_1608Metric, symbol Device:R
- added R36: 82k, Resistor_SMD:R_0603_1608Metric, symbol Device:R
- added R37, R42: 330, Resistor_SMD:R_0603_1608Metric, symbol Device:R
- added R38, R44: 10k, Resistor_SMD:R_0603_1608Metric, symbol Device:R
- added R39, R43: DNP (10k), Resistor_SMD:R_0603_1608Metric, symbol Device:R
- added R41: 0, Resistor_SMD:R_0603_1608Metric, symbol Device:R
- added U7: MCP6002, Package_SO:SOIC-8_3.9x4.9mm_P1.27mm, symbol Amplifier_Operational:MCP6002-xMS
Connections:
- net +5V: now also C28.2, R38.2, R43.2, U7.8 (V+)
- net GND: now also C28.1, R35.1, R39.1, R40.1, R44.1, U7.4 (V-)
- new net: R35.2, R36.1, U7.2 (-)
- new net: R40.2, R41.1, U7.6 (-)
- new net: R36.2, R37.1, U7.1
- new net: R41.2, R42.1, U7.7
- new net DAC1: U7.3 (+)
- new net DAC1_OUT: J40.1 (Pin_1), R37.2, R38.1, R39.2
- new net DAC2: U7.5 (+)
- new net DAC2_OUT: J40.2 (Pin_2), R42.2, R43.1, R44.2
Other:
- note added: "Gain ratio - 1.0"
- note added: "Gain ratio - 1.524"

Commit message: V2.5 with OPAmp
Parts:
- added R45: 120, Resistor_SMD:R_0805_2012Metric, symbol Device:R
Connections:
- net CAN_H: now also R45.1
- net CAN_L: now also R45.2
Changed lines of the file:
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@@
     (comment 1 "STM32F072CBT6")
   )
-  (junction (at 77.47 49.53) (diameter 0) (color 0 0 0 0)
-  )
   (junction (at 116.84 114.3) (diameter 0) (color 0 0 0 0)
   )
@@
   (junction (at 107.95 172.085) (diameter 0) (color 0 0 0 0)
   )
+  (junction (at 77.47 42.545) (diameter 0) (color 0 0 0 0)
+  )
   (junction (at 153.67 35.56) (diameter 0) (color 0 0 0 0)
   )
-  (junction (at 77.47 44.45) (diameter 0) (color 0 0 0 0)
-  )
   (junction (at 46.355 151.13) (diameter 0) (color 0 0 0 0)
   )
@@
   )
   (junction (at 145.415 35.56) (diameter 0) (color 0 0 0 0)
+  )
+  (junction (at 77.47 51.435) (diameter 0) (color 0 0 0 0)
   )
   (junction (at 61.595 148.59) (diameter 0) (color 0 0 0 0)
@@
     (stroke (width 0) (type default) (color 0 0 0 0))
   )
-  (wire (pts (xy 86.36 49.53) (xy 77.47 49.53))
+  (wire (pts (xy 71.755 42.545) (xy 77.47 42.545))
     (stroke (width 0) (type default) (color 0 0 0 0))
   )
@@
     (stroke (width 0) (type default) (color 0 0 0 0))
   )
+  (wire (pts (xy 71.755 51.435) (xy 77.47 51.435))
+    (stroke (width 0) (type default) (color 0 0 0 0))
+  )
   (wire (pts (xy 214.63 33.655) (xy 228.6 33.655))
     (stroke (width 0) (type default) (color 0 0 0 0))
@@
     (stroke (width 0) (type default) (color 0 0 0 0))
   )
+  (wire (pts (xy 71.755 49.53) (xy 71.755 51.435))
+    (stroke (width 0) (type default) (color 0 0 0 0))
+  )
   (wire (pts (xy 111.76 43.815) (xy 111.76 48.26))
     (stroke (width 0) (type default) (color 0 0 0 0))
@@
     (stroke (width 0) (type default) (color 0 0 0 0))
   )
-  (wire (pts (xy 77.47 49.53) (xy 77.47 52.07))
-    (stroke (width 0) (type default) (color 0 0 0 0))
-  )
   (wire (pts (xy 61.595 158.115) (xy 61.595 148.59))
     (stroke (width 0) (type default) (color 0 0 0 0))
@@
     (stroke (width 0) (type default) (color 0 0 0 0))
   )
-  (wire (pts (xy 86.36 44.45) (xy 77.47 44.45))
-    (stroke (width 0) (type default) (color 0 0 0 0))
-  )
   (wire (pts (xy 242.57 103.505) (xy 252.095 103.505))
     (stroke (width 0) (type default) (color 0 0 0 0))
@@
     (stroke (width 0) (type default) (color 0 0 0 0))
   )
-  (wire (pts (xy 77.47 44.45) (xy 71.755 44.45))
-    (stroke (width 0) (type default) (color 0 0 0 0))
-  )
   (wire (pts (xy 214.63 31.115) (xy 228.6 31.115))
     (stroke (width 0) (type default) (color 0 0 0 0))
@@
     (stroke (width 0) (type default) (color 0 0 0 0))
   )
+  (wire (pts (xy 77.47 51.435) (xy 81.915 51.435))
+    (stroke (width 0) (type default) (color 0 0 0 0))
+  )
   (wire (pts (xy 111.76 57.785) (xy 111.76 55.88))
     (stroke (width 0) (type default) (color 0 0 0 0))
@@
     (stroke (width 0) (type default) (color 0 0 0 0))
   )
-  (wire (pts (xy 77.47 49.53) (xy 71.755 49.53))
-    (stroke (width 0) (type default) (color 0 0 0 0))
-  )
   (wire (pts (xy 116.84 99.06) (xy 122.555 99.06))
     (stroke (width 0) (type default) (color 0 0 0 0))
@@
     (stroke (width 0) (type default) (color 0 0 0 0))
   )
+  (wire (pts (xy 71.755 44.45) (xy 71.755 42.545))
+    (stroke (width 0) (type default) (color 0 0 0 0))
+  )
   (wire (pts (xy 145.415 35.56) (xy 153.67 35.56))
     (stroke (width 0) (type default) (color 0 0 0 0))
@@
     (stroke (width 0) (type default) (color 0 0 0 0))
   )
+  (wire (pts (xy 77.47 51.435) (xy 77.47 52.07))
+    (stroke (width 0) (type default) (color 0 0 0 0))
+  )
   (wire (pts (xy 33.655 44.45) (xy 46.355 44.45))
     (stroke (width 0) (type default) (color 0 0 0 0))
@@
     (stroke (width 0) (type default) (color 0 0 0 0))
   )
-  (wire (pts (xy 77.47 41.91) (xy 77.47 44.45))
+  (wire (pts (xy 77.47 41.91) (xy 77.47 42.545))
     (stroke (width 0) (type default) (color 0 0 0 0))
   )
@@
     (stroke (width 0) (type default) (color 0 0 0 0))
   )
+  (wire (pts (xy 77.47 42.545) (xy 81.915 42.545))
+    (stroke (width 0) (type default) (color 0 0 0 0))
+  )
   (wire (pts (xy 77.47 180.34) (xy 77.47 181.61))
     (stroke (width 0) (type default) (color 0 0 0 0))
@@
     (stroke (width 0) (type default) (color 0 0 0 0))
   )
+  (wire (pts (xy 77.47 42.545) (xy 77.47 43.18))
+    (stroke (width 0) (type default) (color 0 0 0 0))
+  )
   (wire (pts (xy 57.785 189.865) (xy 61.595 189.865))
     (stroke (width 0) (type default) (color 0 0 0 0))
   )
   (wire (pts (xy 57.15 158.115) (xy 61.595 158.115))
+    (stroke (width 0) (type default) (color 0 0 0 0))
+  )
+  (wire (pts (xy 77.47 50.8) (xy 77.47 51.435))
     (stroke (width 0) (type default) (color 0 0 0 0))
   )
@@
     (effects (font (size 1.27 1.27) (thickness 0.254) bold) (justify right bottom))
   )
-  (label "CAN_L" (at 86.36 49.53 180)
-    (effects (font (size 1.27 1.27)) (justify right bottom))
+  (label "CAN_L" (at 81.915 51.435 0)
+    (effects (font (size 1.27 1.27)) (justify left bottom))
   )
   (label "LSU_Heater+" (at 241.935 53.975 0)
@@
     (effects (font (size 1.27 1.27)) (justify left bottom))
   )
-  (label "CAN_H" (at 86.36 44.45 180)
-    (effects (font (size 1.27 1.27)) (justify right bottom))
+  (label "CAN_H" (at 81.915 42.545 0)
+    (effects (font (size 1.27 1.27)) (justify left bottom))
   )
   (label "GND" (at 229.87 103.505 180)
@@
       (effects (font (size 1.27 1.27)) hide)
     )
+    (pin "1")
+    (pin "2")
+  )
+  (symbol (lib_id "Device:R") (at 77.47 46.99 0) (unit 1)
+    (in_bom yes) (on_board yes) (fields_autoplaced)
+    (property "Reference" "R45" (id 0) (at 79.248 46.1553 0)
+      (effects (font (size 1.27 1.27)) (justify left))
+    )
+    (property "Value" "120" (id 1) (at 79.248 48.6922 0)
+      (effects (font (size 1.27 1.27)) (justify left))
+    )
+    (property "Footprint" "Resistor_SMD:R_0805_2012Metric" (id 2) (at 75.692 46.99 90)
+      (effects (font (size 1.27 1.27)) hide)
+    )
+    (property "Datasheet" "~" (id 3) (at 77.47 46.99 0)
+      (effects (font (size 1.27 1.27)) hide)
+    )

Commit message: V2.5 with OPAmp
Parts:
- R40: value 160k -> 100k
Connections:
- net DAC2: now also U7.6 (-); no longer U7.5 (+)
- net at R40.2, R41.1: now also U7.5 (+); no longer U7.6 (-)
Other:
- moved on the sheet: R40, R41
Changed lines of the file:
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@@
   (title_block
     (title "MRE addon board V2- WBO2 & EGT & SD Card")
-    (date "2023-01-23")
+    (date "2023-01-31")
     (rev "V2.5")
     (company "by JRD McLAREN")
@@
   (junction (at 116.84 114.3) (diameter 0) (color 0 0 0 0)
   )
-  (junction (at 46.355 182.88) (diameter 0) (color 0 0 0 0)
+  (junction (at 46.355 177.8) (diameter 0) (color 0 0 0 0)
   )
   (junction (at 107.95 156.845) (diameter 0) (color 0 0 0 0)
   )
+  (junction (at 77.47 180.34) (diameter 0) (color 0 0 0 0)
+  )
+  (junction (at 107.95 172.085) (diameter 0) (color 0 0 0 0)
+  )
+  (junction (at 77.47 42.545) (diameter 0) (color 0 0 0 0)
+  )
+  (junction (at 153.67 35.56) (diameter 0) (color 0 0 0 0)
+  )
+  (junction (at 46.355 151.13) (diameter 0) (color 0 0 0 0)
+  )
   (junction (at 61.595 180.34) (diameter 0) (color 0 0 0 0)
-  )
-  (junction (at 77.47 180.34) (diameter 0) (color 0 0 0 0)
-  )
-  (junction (at 107.95 172.085) (diameter 0) (color 0 0 0 0)
-  )
-  (junction (at 77.47 42.545) (diameter 0) (color 0 0 0 0)
-  )
-  (junction (at 153.67 35.56) (diameter 0) (color 0 0 0 0)
-  )
-  (junction (at 46.355 151.13) (diameter 0) (color 0 0 0 0)
   )
   (junction (at 116.84 99.06) (diameter 0) (color 0 0 0 0)
@@
   (no_connect (at 36.83 99.06))
   (no_connect (at 242.57 106.045))
-  (wire (pts (xy 46.355 189.865) (xy 50.165 189.865))
+  (wire (pts (xy 46.355 173.99) (xy 50.165 173.99))
     (stroke (width 0) (type default) (color 0 0 0 0))
   )
@@
     (stroke (width 0) (type default) (color 0 0 0 0))
   )
-  (wire (pts (xy 38.735 182.88) (xy 38.735 189.865))
-    (stroke (width 0) (type default) (color 0 0 0 0))
-  )
   (wire (pts (xy 77.47 146.685) (xy 77.47 148.59))
     (stroke (width 0) (type default) (color 0 0 0 0))
@@
     (stroke (width 0) (type default) (color 0 0 0 0))
   )
-  (wire (pts (xy 38.735 151.13) (xy 38.735 158.115))
+  (wire (pts (xy 38.735 151.13) (xy 33.02 151.13))
     (stroke (width 0) (type default) (color 0 0 0 0))
   )
@@
     (stroke (width 0) (type default) (color 0 0 0 0))
   )
+  (wire (pts (xy 46.355 173.99) (xy 46.355 177.8))
+    (stroke (width 0) (type default) (color 0 0 0 0))
+  )
   (wire (pts (xy 101.6 156.845) (xy 107.95 156.845))
     (stroke (width 0) (type default) (color 0 0 0 0))
@@
     (stroke (width 0) (type default) (color 0 0 0 0))
   )
+  (wire (pts (xy 33.655 177.8) (xy 38.735 177.8))
+    (stroke (width 0) (type default) (color 0 0 0 0))
+  )
   (wire (pts (xy 114.3 36.195) (xy 106.68 36.195))
     (stroke (width 0) (type default) (color 0 0 0 0))
@@
     (stroke (width 0) (type default) (color 0 0 0 0))
   )
-  (wire (pts (xy 46.355 182.88) (xy 46.355 189.865))
-    (stroke (width 0) (type default) (color 0 0 0 0))
-  )
   (wire (pts (xy 227.965 60.325) (xy 237.49 60.325))
     (stroke (width 0) (type default) (color 0 0 0 0))
@@
     (stroke (width 0) (type default) (color 0 0 0 0))
   )
+  (wire (pts (xy 33.655 182.88) (xy 46.355 182.88))
+    (stroke (width 0) (type default) (color 0 0 0 0))
+  )
   (wire (pts (xy 222.25 103.505) (xy 229.87 103.505))
     (stroke (width 0) (type default) (color 0 0 0 0))
@@
     (stroke (width 0) (type default) (color 0 0 0 0))
   )
-  (wire (pts (xy 61.595 189.865) (xy 61.595 180.34))
-    (stroke (width 0) (type default) (color 0 0 0 0))
-  )
   (wire (pts (xy 242.57 95.885) (xy 252.095 95.885))
     (stroke (width 0) (type default) (color 0 0 0 0))
@@
     (stroke (width 0) (type default) (color 0 0 0 0))
   )
-  (wire (pts (xy 33.02 177.8) (xy 46.355 177.8))
-    (stroke (width 0) (type default) (color 0 0 0 0))
-  )
   (wire (pts (xy 242.57 98.425) (xy 252.095 98.425))
     (stroke (width 0) (type default) (color 0 0 0 0))
@@
     (stroke (width 0) (type default) (color 0 0 0 0))
   )
-  (wire (pts (xy 57.785 189.865) (xy 61.595 189.865))
+  (wire (pts (xy 57.785 173.99) (xy 61.595 173.99))
     (stroke (width 0) (type default) (color 0 0 0 0))
   )
@@
   )
   (wire (pts (xy 116.84 114.3) (xy 122.555 114.3))
+    (stroke (width 0) (type default) (color 0 0 0 0))
+  )
+  (wire (pts (xy 61.595 173.99) (xy 61.595 180.34))
     (stroke (width 0) (type default) (color 0 0 0 0))
   )
@@
     )
   )
-  (global_label "DAC2" (shape input) (at 33.02 177.8 180) (fields_autoplaced)
+  (global_label "DAC2" (shape input) (at 33.655 182.88 180) (fields_autoplaced)
     (effects (font (size 1.27 1.27)) (justify right))
-    (property "Medzirezortné odkazy" "${INTERSHEET_REFS}" (id 0) (at 25.8577 177.7206 0)
+    (property "Medzirezortné odkazy" "${INTERSHEET_REFS}" (id 0) (at 26.4927 182.8006 0)
       (effects (font (size 1.27 1.27)) (justify right) hide)
     )
@@
     (pin "2")
   )
-  (symbol (lib_id "power:GND") (at 38.735 158.115 0) (unit 1)
-    (in_bom yes) (on_board yes) (fields_autoplaced)
-    (property "Reference" "#PWR0180" (id 0) (at 38.735 164.465 0)
-      (effects (font (size 1.27 1.27)) hide)
-    )
-    (property "Value" "GND" (id 1) (at 38.735 162.5584 0))
-    (property "Footprint" "" (id 2) (at 38.735 158.115 0)
-      (effects (font (size 1.27 1.27)) hide)
-    )
-    (property "Datasheet" "" (id 3) (at 38.735 158.115 0)
+  (symbol (lib_id "power:GND") (at 33.02 151.13 270) (unit 1)
+    (in_bom yes) (on_board yes) (fields_autoplaced)
+    (property "Reference" "#PWR0180" (id 0) (at 26.67 151.13 0)
+      (effects (font (size 1.27 1.27)) hide)
+    )
+    (property "Value" "GND" (id 1) (at 29.8451 151.5638 90)
+      (effects (font (size 1.27 1.27)) (justify right))
+    )
+    (property "Footprint" "" (id 2) (at 33.02 151.13 0)
+      (effects (font (size 1.27 1.27)) hide)
+    )
+    (property "Datasheet" "" (id 3) (at 33.02 151.13 0)
       (effects (font (size 1.27 1.27)) hide)
     )
@@
     (pin "1")
   )
-  (symbol (lib_id "Device:R") (at 42.545 182.88 90) (unit 1)
-    (in_bom yes) (on_board yes) (fields_autoplaced)
-    (property "Reference" "R40" (id 0) (at 42.545 187.5958 90))
-    (property "Value" "160k" (id 1) (at 42.545 185.0589 90))
-    (property "Footprint" "Resistor_SMD:R_0603_1608Metric" (id 2) (at 42.545 184.658 90)
-      (effects (font (size 1.27 1.27)) hide)
-    )
-    (property "Datasheet" "~" (id 3) (at 42.545 182.88 0)
+  (symbol (lib_id "Device:R") (at 42.545 177.8 90) (unit 1)
+    (in_bom yes) (on_board yes)
+    (property "Reference" "R40" (id 0) (at 42.545 175.26 90))
+    (property "Value" "100k" (id 1) (at 42.545 179.9789 90))
+    (property "Footprint" "Resistor_SMD:R_0603_1608Metric" (id 2) (at 42.545 179.578 90)
+      (effects (font (size 1.27 1.27)) hide)
+    )
+    (property "Datasheet" "~" (id 3) (at 42.545 177.8 0)
       (effects (font (size 1.27 1.27)) hide)
     )
@@
     (pin "1")
   )
-  (symbol (lib_id "power:GND") (at 38.735 189.865 0) (unit 1)
-    (in_bom yes) (on_board yes) (fields_autoplaced)
-    (property "Reference" "#PWR0179" (id 0) (at 38.735 196.215 0)
-      (effects (font (size 1.27 1.27)) hide)
-    )
-    (property "Value" "GND" (id 1) (at 38.735 194.3084 0))
-    (property "Footprint" "" (id 2) (at 38.735 189.865 0)
-      (effects (font (size 1.27 1.27)) hide)
-    )
-    (property "Datasheet" "" (id 3) (at 38.735 189.865 0)
+  (symbol (lib_id "power:GND") (at 33.655 177.8 270) (unit 1)
+    (in_bom yes) (on_board yes) (fields_autoplaced)
+    (property "Reference" "#PWR0179" (id 0) (at 27.305 177.8 0)
+      (effects (font (size 1.27 1.27)) hide)
+    )
+    (property "Value" "GND" (id 1) (at 30.4801 178.2338 90)
+      (effects (font (size 1.27 1.27)) (justify right))
+    )
+    (property "Footprint" "" (id 2) (at 33.655 177.8 0)
+      (effects (font (size 1.27 1.27)) hide)
+    )
+    (property "Datasheet" "" (id 3) (at 33.655 177.8 0)
       (effects (font (size 1.27 1.27)) hide)
     )
@@
   )
   (symbol (lib_id "Amplifier_Operational:MCP6002-xMS") (at 53.975 180.34 0) (unit 2)
-    (in_bom yes) (on_board yes) (fields_autoplaced)
-    (property "Reference" "U7" (id 0) (at 53.975 171.5602 0))
-    (property "Value" "MCP6002" (id 1) (at 53.975 174.0971 0))
+    (in_bom yes) (on_board yes)
+    (property "Reference" "U7" (id 0) (at 53.975 187.325 0))
+    (property "Value" "MCP6002" (id 1) (at 53.975 189.865 0))
     (property "Footprint" "Package_SO:SOIC-8_3.9x4.9mm_P1.27mm" (id 2) (at 53.975 180.34 0)
       (effects (font (size 1.27 1.27)) hide)
@@
     (pin "8")
   )
-  (symbol (lib_id "Device:R") (at 53.975 189.865 90) (unit 1)
-    (in_bom yes) (on_board yes) (fields_autoplaced)
-    (property "Reference" "R41" (id 0) (at 53.975 185.1492 90))
-    (property "Value" "0" (id 1) (at 53.975 187.6861 90))
-    (property "Footprint" "Resistor_SMD:R_0603_1608Metric" (id 2) (at 53.975 191.643 90)
-      (effects (font (size 1.27 1.27)) hide)
-    )
-    (property "Datasheet" "~" (id 3) (at 53.975 189.865 0)
-      (effects (font (size 1.27 1.27)) hide)
-    )
+  (symbol (lib_id "Device:R") (at 53.975 173.99 90) (unit 1)
+    (in_bom yes) (on_board yes) (fields_autoplaced)
+    (property "Reference" "R41" (id 0) (at 53.975 169.2742 90))
+    (property "Value" "0" (id 1) (at 53.975 171.8111 90))
+    (property "Footprint" "Resistor_SMD:R_0603_1608Metric" (id 2) (at 53.975 175.768 90)
+      (effects (font (size 1.27 1.27)) hide)
+    )
+    (property "Datasheet" "~" (id 3) (at 53.975 173.99 0)
+      (effects (font (size 1.27 1.27)) hide)
+    )
