File: can_fet_egt_sd_v2.kicad_sch (KiCad schematic)
At the start: 35 parts, among them J10 Molex_Micro-Fit_3.0_43045-080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, J15 microSD_HC_Wuerth_693072010801, J20 Conn_02x05_Odd_Even-Connector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, J21 Soldering PAD for 12V_MREL, J30 Conn_02x05_Odd_Even-Connector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, J40 Molex_Micro-Fit_3.0_43045-020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, J41 CONN_Sparkfun, Q1 BTS3028, U5 TJA1051T-3, U6 MAX31855KASA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

Commit message: some changes on DAC pins
Connections:
- net DAC1: now also U7.6 (-); no longer U7.3 (+)
- net DAC1_OUT: now also R42.2, R43.1, R44.2; no longer R37.2, R38.1, R39.2
- net DAC2: now also U7.3 (+); no longer U7.6 (-)
- net DAC2_OUT: now also R37.2, R38.1, R39.2; no longer R42.2, R43.1, R44.2
Changed lines of the file:
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@@
   (title_block
     (title "MRE addon board V2- WBO2 & EGT & SD Card")
-    (date "2023-01-31")
+    (date "2023-02-05")
     (rev "V2.5")
     (company "by JRD McLAREN")
@@
     (stroke (width 0) (type default) (color 0 0 0 0))
   )
+  (wire (pts (xy 81.28 123.19) (xy 81.28 121.92))
+    (stroke (width 0) (type default) (color 0 0 0 0))
+  )
+  (wire (pts (xy 91.44 97.79) (xy 91.44 102.235))
+    (stroke (width 0) (type default) (color 0 0 0 0))
+  )
+  (wire (pts (xy 46.355 158.115) (xy 49.53 158.115))
+    (stroke (width 0) (type default) (color 0 0 0 0))
+  )
+  (wire (pts (xy 172.72 30.48) (xy 172.72 27.305))
+    (stroke (width 0) (type default) (color 0 0 0 0))
+  )
+  (wire (pts (xy 71.755 51.435) (xy 77.47 51.435))
+    (stroke (width 0) (type default) (color 0 0 0 0))
+  )
+  (wire (pts (xy 214.63 33.655) (xy 228.6 33.655))
+    (stroke (width 0) (type default) (color 0 0 0 0))
+  )
+  (wire (pts (xy 238.76 53.975) (xy 241.935 53.975))
+    (stroke (width 0) (type default) (color 0 0 0 0))
+  )
+  (wire (pts (xy 116.84 110.49) (xy 116.84 114.3))
+    (stroke (width 0) (type default) (color 0 0 0 0))
+  )
+  (wire (pts (xy 38.735 151.13) (xy 33.02 151.13))
+    (stroke (width 0) (type default) (color 0 0 0 0))
+  )
+  (wire (pts (xy 74.93 180.34) (xy 77.47 180.34))
+    (stroke (width 0) (type default) (color 0 0 0 0))
+  )
+  (wire (pts (xy 228.6 36.195) (xy 214.63 36.195))
+    (stroke (width 0) (type default) (color 0 0 0 0))
+  )
+  (wire (pts (xy 74.93 148.59) (xy 77.47 148.59))
+    (stroke (width 0) (type default) (color 0 0 0 0))
+  )
+  (wire (pts (xy 46.355 173.99) (xy 46.355 177.8))
+    (stroke (width 0) (type default) (color 0 0 0 0))
+  )
+  (wire (pts (xy 101.6 156.845) (xy 107.95 156.845))
+    (stroke (width 0) (type default) (color 0 0 0 0))
+  )
+  (wire (pts (xy 67.31 180.34) (xy 61.595 180.34))
+    (stroke (width 0) (type default) (color 0 0 0 0))
+  )
+  (wire (pts (xy 241.3 31.115) (xy 255.27 31.115))
+    (stroke (width 0) (type default) (color 0 0 0 0))
+  )
+  (wire (pts (xy 71.755 49.53) (xy 71.755 51.435))
+    (stroke (width 0) (type default) (color 0 0 0 0))
+  )
+  (wire (pts (xy 111.76 43.815) (xy 111.76 48.26))
+    (stroke (width 0) (type default) (color 0 0 0 0))
+  )
+  (wire (pts (xy 122.555 99.06) (xy 122.555 106.68))
+    (stroke (width 0) (type default) (color 0 0 0 0))
+  )
+  (wire (pts (xy 252.095 103.505) (xy 252.095 110.49))
+    (stroke (width 0) (type default) (color 0 0 0 0))
+  )
+  (wire (pts (xy 227.965 53.975) (xy 231.14 53.975))
+    (stroke (width 0) (type default) (color 0 0 0 0))
+  )
+  (wire (pts (xy 116.84 102.87) (xy 116.84 99.06))
+    (stroke (width 0) (type default) (color 0 0 0 0))
+  )
+  (wire (pts (xy 33.655 177.8) (xy 38.735 177.8))
+    (stroke (width 0) (type default) (color 0 0 0 0))
+  )
+  (wire (pts (xy 114.3 36.195) (xy 106.68 36.195))
+    (stroke (width 0) (type default) (color 0 0 0 0))
+  )
+  (wire (pts (xy 91.44 111.76) (xy 91.44 109.855))
+    (stroke (width 0) (type default) (color 0 0 0 0))
+  )
   (wire (pts (xy 77.47 148.59) (xy 85.725 148.59))
     (stroke (width 0) (type default) (color 0 0 0 0))
   )
-  (wire (pts (xy 81.28 123.19) (xy 81.28 121.92))
-    (stroke (width 0) (type default) (color 0 0 0 0))
-  )
-  (wire (pts (xy 91.44 97.79) (xy 91.44 102.235))
-    (stroke (width 0) (type default) (color 0 0 0 0))
-  )
-  (wire (pts (xy 46.355 158.115) (xy 49.53 158.115))
-    (stroke (width 0) (type default) (color 0 0 0 0))
-  )
-  (wire (pts (xy 172.72 30.48) (xy 172.72 27.305))
-    (stroke (width 0) (type default) (color 0 0 0 0))
-  )
-  (wire (pts (xy 71.755 51.435) (xy 77.47 51.435))
-    (stroke (width 0) (type default) (color 0 0 0 0))
-  )
-  (wire (pts (xy 214.63 33.655) (xy 228.6 33.655))
-    (stroke (width 0) (type default) (color 0 0 0 0))
-  )
-  (wire (pts (xy 238.76 53.975) (xy 241.935 53.975))
-    (stroke (width 0) (type default) (color 0 0 0 0))
-  )
-  (wire (pts (xy 116.84 110.49) (xy 116.84 114.3))
-    (stroke (width 0) (type default) (color 0 0 0 0))
-  )
-  (wire (pts (xy 38.735 151.13) (xy 33.02 151.13))
-    (stroke (width 0) (type default) (color 0 0 0 0))
-  )
-  (wire (pts (xy 74.93 180.34) (xy 77.47 180.34))
-    (stroke (width 0) (type default) (color 0 0 0 0))
-  )
-  (wire (pts (xy 228.6 36.195) (xy 214.63 36.195))
-    (stroke (width 0) (type default) (color 0 0 0 0))
-  )
-  (wire (pts (xy 74.93 148.59) (xy 77.47 148.59))
-    (stroke (width 0) (type default) (color 0 0 0 0))
-  )
-  (wire (pts (xy 46.355 173.99) (xy 46.355 177.8))
-    (stroke (width 0) (type default) (color 0 0 0 0))
-  )
-  (wire (pts (xy 101.6 156.845) (xy 107.95 156.845))
-    (stroke (width 0) (type default) (color 0 0 0 0))
-  )
-  (wire (pts (xy 67.31 180.34) (xy 61.595 180.34))
-    (stroke (width 0) (type default) (color 0 0 0 0))
-  )
-  (wire (pts (xy 241.3 31.115) (xy 255.27 31.115))
-    (stroke (width 0) (type default) (color 0 0 0 0))
-  )
-  (wire (pts (xy 71.755 49.53) (xy 71.755 51.435))
-    (stroke (width 0) (type default) (color 0 0 0 0))
-  )
-  (wire (pts (xy 111.76 43.815) (xy 111.76 48.26))
-    (stroke (width 0) (type default) (color 0 0 0 0))
-  )
-  (wire (pts (xy 122.555 99.06) (xy 122.555 106.68))
-    (stroke (width 0) (type default) (color 0 0 0 0))
-  )
-  (wire (pts (xy 252.095 103.505) (xy 252.095 110.49))
-    (stroke (width 0) (type default) (color 0 0 0 0))
-  )
-  (wire (pts (xy 227.965 53.975) (xy 231.14 53.975))
-    (stroke (width 0) (type default) (color 0 0 0 0))
-  )
-  (wire (pts (xy 116.84 102.87) (xy 116.84 99.06))
-    (stroke (width 0) (type default) (color 0 0 0 0))
-  )
-  (wire (pts (xy 33.655 177.8) (xy 38.735 177.8))
-    (stroke (width 0) (type default) (color 0 0 0 0))
-  )
-  (wire (pts (xy 114.3 36.195) (xy 106.68 36.195))
-    (stroke (width 0) (type default) (color 0 0 0 0))
-  )
-  (wire (pts (xy 77.47 180.34) (xy 86.36 180.34))
-    (stroke (width 0) (type default) (color 0 0 0 0))
-  )
-  (wire (pts (xy 91.44 111.76) (xy 91.44 109.855))
-    (stroke (width 0) (type default) (color 0 0 0 0))
-  )
   (wire (pts (xy 101.6 167.64) (xy 101.6 172.085))
     (stroke (width 0) (type default) (color 0 0 0 0))
@@
     (stroke (width 0) (type default) (color 0 0 0 0))
   )
-  (wire (pts (xy 33.655 182.88) (xy 46.355 182.88))
-    (stroke (width 0) (type default) (color 0 0 0 0))
-  )
   (wire (pts (xy 222.25 103.505) (xy 229.87 103.505))
     (stroke (width 0) (type default) (color 0 0 0 0))
@@
     (stroke (width 0) (type default) (color 0 0 0 0))
   )
+  (wire (pts (xy 77.47 180.34) (xy 85.725 180.34))
+    (stroke (width 0) (type default) (color 0 0 0 0))
+  )
   (wire (pts (xy 242.57 95.885) (xy 252.095 95.885))
     (stroke (width 0) (type default) (color 0 0 0 0))
@@
     (stroke (width 0) (type default) (color 0 0 0 0))
   )
-  (wire (pts (xy 33.02 146.05) (xy 46.355 146.05))
-    (stroke (width 0) (type default) (color 0 0 0 0))
-  )
   (wire (pts (xy 71.755 44.45) (xy 71.755 42.545))
     (stroke (width 0) (type default) (color 0 0 0 0))
@@
     (stroke (width 0) (type default) (color 0 0 0 0))
   )
+  (wire (pts (xy 32.385 182.88) (xy 46.355 182.88))
+    (stroke (width 0) (type default) (color 0 0 0 0))
+  )
   (wire (pts (xy 33.655 44.45) (xy 46.355 44.45))
     (stroke (width 0) (type default) (color 0 0 0 0))
@@
   )
   (wire (pts (xy 77.47 50.8) (xy 77.47 51.435))
+    (stroke (width 0) (type default) (color 0 0 0 0))
+  )
+  (wire (pts (xy 31.75 146.05) (xy 46.355 146.05))
     (stroke (width 0) (type default) (color 0 0 0 0))
   )
@@
     (effects (font (size 1.27 1.27)) (justify left bottom))
   )
-  (label "DAC2_OUT" (at 86.36 180.34 0)
+  (label "DAC2_OUT" (at 85.725 148.59 0)
     (effects (font (size 1.27 1.27)) (justify left bottom))
   )
@@
     (effects (font (size 1.27 1.27)) (justify right bottom))
   )
-  (label "DAC1_OUT" (at 85.725 148.59 0)
+  (label "DAC1_OUT" (at 85.725 180.34 0)
     (effects (font (size 1.27 1.27)) (justify left bottom))
   )
@@
     )
   )
-  (global_label "DAC1" (shape input) (at 33.02 146.05 180) (fields_autoplaced)
-    (effects (font (size 1.27 1.27)) (justify right))
-    (property "Medzirezortné odkazy" "${INTERSHEET_REFS}" (id 0) (at 25.8577 145.9706 0)
+  (global_label "DAC1" (shape input) (at 32.385 182.88 180) (fields_autoplaced)
+    (effects (font (size 1.27 1.27)) (justify right))
+    (property "Medzirezortné odkazy" "${INTERSHEET_REFS}" (id 0) (at 25.2227 182.8006 0)
       (effects (font (size 1.27 1.27)) (justify right) hide)
     )
@@
     )
   )
-  (global_label "DAC2" (shape input) (at 33.655 182.88 180) (fields_autoplaced)
-    (effects (font (size 1.27 1.27)) (justify right))
-    (property "Medzirezortné odkazy" "${INTERSHEET_REFS}" (id 0) (at 26.4927 182.8006 0)
+  (global_label "DAC2" (shape input) (at 31.75 146.05 180) (fields_autoplaced)
+    (effects (font (size 1.27 1.27)) (justify right))
+    (property "Medzirezortné odkazy" "${INTERSHEET_REFS}" (id 0) (at 24.5877 145.9706 0)
       (effects (font (size 1.27 1.27)) (justify right) hide)
     )
