File: mre_addon_v2.kicad_sch (KiCad schematic)
At the start: 0 parts

Commit message: V2.5 with OPAmp
Changed lines of the file:
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@@
   (title_block
     (title "MRE addon board V2- WBO2 & EGT & SD Card")
-    (date "2023-01-06")
+    (date "2023-01-23")
     (rev "V2.5")
     (company "by JRD McLAREN")
@@
     (stroke (width 0) (type default) (color 0 0 0 0))
   )
+  (wire (pts (xy 131.445 84.455) (xy 150.495 84.455))
+    (stroke (width 0) (type default) (color 0 0 0 0))
+  )
   (wire (pts (xy 131.445 106.045) (xy 150.495 106.045))
     (stroke (width 0) (type default) (color 0 0 0 0))
@@
     (stroke (width 0) (type default) (color 0 0 0 0))
   )
+  (wire (pts (xy 131.445 86.995) (xy 150.495 86.995))
+    (stroke (width 0) (type default) (color 0 0 0 0))
+  )
   (wire (pts (xy 131.445 76.2) (xy 150.495 76.2))
     (stroke (width 0) (type default) (color 0 0 0 0))
@@
     )
   )
+  (global_label "DAC1" (shape input) (at 150.495 84.455 0) (fields_autoplaced)
+    (effects (font (size 1.27 1.27)) (justify left))
+    (property "Medzirezortné odkazy" "${INTERSHEET_REFS}" (id 0) (at 157.6573 84.3756 0)
+      (effects (font (size 1.27 1.27)) (justify left) hide)
+    )
+  )
+  (global_label "DAC1" (shape input) (at 131.445 84.455 180) (fields_autoplaced)
+    (effects (font (size 1.27 1.27)) (justify right))
+    (property "Medzirezortné odkazy" "${INTERSHEET_REFS}" (id 0) (at 124.2827 84.3756 0)
+      (effects (font (size 1.27 1.27)) (justify right) hide)
+    )
+  )
   (global_label "GND" (shape input) (at 131.445 108.585 180) (fields_autoplaced)
     (effects (font (size 1.27 1.27)) (justify right))
@@
     )
   )
+  (global_label "DAC2" (shape input) (at 150.495 86.995 0) (fields_autoplaced)
+    (effects (font (size 1.27 1.27)) (justify left))
+    (property "Medzirezortné odkazy" "${INTERSHEET_REFS}" (id 0) (at 157.6573 86.9156 0)
+      (effects (font (size 1.27 1.27)) (justify left) hide)
+    )
+  )
   (global_label "LSU_Un" (shape input) (at 150.495 73.66 0) (fields_autoplaced)
     (effects (font (size 1.27 1.27)) (justify left))
@@
     (property "Medzirezortné odkazy" "${INTERSHEET_REFS}" (id 0) (at 0 0 0)
       (effects (font (size 1.27 1.27)) hide)
+    )
+  )
+  (global_label "DAC2" (shape input) (at 131.445 86.995 180) (fields_autoplaced)
+    (effects (font (size 1.27 1.27)) (justify right))
+    (property "Medzirezortné odkazy" "${INTERSHEET_REFS}" (id 0) (at 124.2827 86.9156 0)
+      (effects (font (size 1.27 1.27)) (justify right) hide)
     )
   )
@@
       (reference "#PWR0176") (unit 1) (value "GND-power") (footprint "")
     )
+    (path "/00000000-0000-0000-0000-000061a546df/b76d5fa0-0b48-4498-acc2-bfccdd554761"
+      (reference "#PWR0177") (unit 1) (value "GND") (footprint "")
+    )
+    (path "/00000000-0000-0000-0000-000061a546df/7363dd15-612e-4762-b6f6-e1ba8051ac0c"
+      (reference "#PWR0178") (unit 1) (value "+5V") (footprint "")
+    )
+    (path "/00000000-0000-0000-0000-000061a546df/8f54db08-c91d-4388-b220-abc1cc7b9d81"
+      (reference "#PWR0179") (unit 1) (value "GND") (footprint "")
+    )
+    (path "/00000000-0000-0000-0000-000061a546df/1e19935d-b9c5-49ae-a896-1c50baa90914"
+      (reference "#PWR0180") (unit 1) (value "GND") (footprint "")
+    )
+    (path "/00000000-0000-0000-0000-000061a546df/343aa974-168a-41b0-a014-50c69125785e"
+      (reference "#PWR0181") (unit 1) (value "+5V") (footprint "")
+    )
+    (path "/00000000-0000-0000-0000-000061a546df/066bffdc-3461-4699-abbe-83429021df83"
+      (reference "#PWR0182") (unit 1) (value "+5V") (footprint "")
+    )
+    (path "/00000000-0000-0000-0000-000061a546df/ae1f59c0-cb8f-423f-b304-fd059c7071dd"
+      (reference "#PWR0183") (unit 1) (value "GND") (footprint "")
+    )
+    (path "/00000000-0000-0000-0000-000061a546df/8f0677ca-4cb6-40b7-ab62-ac47a2edb874"
+      (reference "#PWR0184") (unit 1) (value "GND") (footprint "")
+    )
+    (path "/00000000-0000-0000-0000-000061a542dd/51cce56c-bbab-4424-81ae-7881e2141a4f"
+      (reference "BOOT_TP1") (unit 1) (value "TestPoint_2Pole") (footprint "TestPoint:TestPoint_Bridge_Pitch2.54mm_Drill0.7mm")
+    )
     (path "/00000000-0000-0000-0000-000061a542dd/00000000-0000-0000-0000-00005eb1294f"
       (reference "C1") (unit 1) (value "1u") (footprint "Capacitor_SMD:C_0603_1608Metric")
@@
       (reference "C27") (unit 1) (value "100nF") (footprint "Capacitor_SMD:C_0603_1608Metric")
     )
+    (path "/00000000-0000-0000-0000-000061a546df/b3bd14af-5444-4717-8499-5b8859f0b1a5"
+      (reference "C28") (unit 1) (value "100n") (footprint "Capacitor_SMD:C_0603_1608Metric")
+    )
     (path "/00000000-0000-0000-0000-000061a546df/00000000-0000-0000-0000-0000618f24c8"
       (reference "C42") (unit 1) (value "100nF") (footprint "Capacitor_SMD:C_0603_1608Metric")
@@
       (reference "J30") (unit 1) (value "Conn_02x05_Odd_Even-Connector_Generic") (footprint "Connector_PinHeader_2.54mm:PinHeader_2x05_P2.54mm_Vertical_SMD")
     )
+    (path "/00000000-0000-0000-0000-000061a546df/9ca6c55b-02a2-4cd2-9a3e-09115a99de15"
+      (reference "J40") (unit 1) (value "Molex_Micro-Fit_3.0_43045-0200_2x01_P3.00mm_Horizontal") (footprint "Molex_Micro-Fit_3.0_43045-0200_2x01_P3.00mm_Horizontal")
+    )
     (path "/00000000-0000-0000-0000-000061a546df/00000000-0000-0000-0000-0000535a15db"
       (reference "J41") (unit 1) (value "CONN_Sparkfun") (footprint "rusefi_lib:tcpl_PCC-SMP")
@@
       (reference "R34") (unit 1) (value "1k") (footprint "Resistor_SMD:R_0603_1608Metric")
     )
-    (path "/00000000-0000-0000-0000-000061a542dd/00000000-0000-0000-0000-000061bd0bc6"
-      (reference "SW1") (unit 1) (value "SW_Push") (footprint "rusefi_lib:SW_SPST_CK_RS282G05A3")
+    (path "/00000000-0000-0000-0000-000061a546df/0b7a76cc-cae1-4a6a-9418-bebb17313168"
+      (reference "R35") (unit 1) (value "160k") (footprint "Resistor_SMD:R_0603_1608Metric")
+    )
+    (path "/00000000-0000-0000-0000-000061a546df/59f94853-1047-476e-8709-e2a66ac18e37"
+      (reference "R36") (unit 1) (value "82k") (footprint "Resistor_SMD:R_0603_1608Metric")
+    )
+    (path "/00000000-0000-0000-0000-000061a546df/c3883a9d-b779-4d76-b87a-9b812f30ef3d"
+      (reference "R37") (unit 1) (value "330") (footprint "Resistor_SMD:R_0603_1608Metric")
+    )
+    (path "/00000000-0000-0000-0000-000061a546df/68bdc370-96f2-40fc-963a-3f4aee58dfd5"
+      (reference "R38") (unit 1) (value "10k") (footprint "Resistor_SMD:R_0603_1608Metric")
+    )
+    (path "/00000000-0000-0000-0000-000061a546df/5946b0c5-b2bd-497b-acb7-6833102db482"
+      (reference "R39") (unit 1) (value "DNP (10k)") (footprint "Resistor_SMD:R_0603_1608Metric")
+    )
+    (path "/00000000-0000-0000-0000-000061a546df/388dfd94-0e6b-4a6d-8988-2ef5bffb269f"
+      (reference "R40") (unit 1) (value "160k") (footprint "Resistor_SMD:R_0603_1608Metric")
+    )
+    (path "/00000000-0000-0000-0000-000061a546df/fe188061-3f94-41b0-a5f7-8d3e50339861"
+      (reference "R41") (unit 1) (value "0") (footprint "Resistor_SMD:R_0603_1608Metric")
+    )
+    (path "/00000000-0000-0000-0000-000061a546df/739c2479-e569-49ed-91e1-d0bccdd497b0"
+      (reference "R42") (unit 1) (value "330") (footprint "Resistor_SMD:R_0603_1608Metric")
+    )
+    (path "/00000000-0000-0000-0000-000061a546df/69a5903a-7a59-4fcb-8b2e-2085893d2336"
+      (reference "R43") (unit 1) (value "DNP (10k)") (footprint "Resistor_SMD:R_0603_1608Metric")
+    )
+    (path "/00000000-0000-0000-0000-000061a546df/b9c88f25-491f-4186-9408-7174947c23c8"
+      (reference "R44") (unit 1) (value "10k") (footprint "Resistor_SMD:R_0603_1608Metric")
     )
     (path "/00000000-0000-0000-0000-000061a542dd/00000000-0000-0000-0000-0000619e9d4b"
@@
       (reference "U6") (unit 1) (value "MAX31855KASA") (footprint "Package_SO:SOIC-8_3.9x4.9mm_P1.27mm")
     )
+    (path "/00000000-0000-0000-0000-000061a546df/cd39e624-e2f4-4e16-9e81-53008133d16f"
+      (reference "U7") (unit 1) (value "MCP6002") (footprint "Package_SO:SOIC-8_3.9x4.9mm_P1.27mm")
+    )
+    (path "/00000000-0000-0000-0000-000061a546df/90b0ad52-f46c-434f-81bb-09780089c4ca"
+      (reference "U7") (unit 2) (value "MCP6002") (footprint "Package_SO:SOIC-8_3.9x4.9mm_P1.27mm")
+    )
+    (path "/00000000-0000-0000-0000-000061a546df/0a04a6c3-461e-47fe-a25d-dbe1ee978eb5"
+      (reference "U7") (unit 3) (value "MCP6002") (footprint "Package_SO:SOIC-8_3.9x4.9mm_P1.27mm")
+    )
     (path "/00000000-0000-0000-0000-000061a542dd/1396927a-5721-4452-b7e0-26ceb9885c8b"
